Commit message: Sim. gripper service

File: fanuc_ros/src/fanuc_lrmate200id_support/urdf/fanuc_lrmate200id.xacro (robot description, xacro)
@@ -22,5 +22,5 @@
             </geometry>
         </collision>
-<inertial>
+        <inertial>
             <mass value="4" />
             <origin rpy="0 0 0" xyz="0 0 0" />
@@ -44,5 +44,5 @@
             </geometry>
         </collision>
-<inertial>
+        <inertial>
             <mass value="4" />
             <origin rpy="0 0 0" xyz="0 0 0" />
@@ -66,5 +66,5 @@
             </geometry>
         </collision>
-<inertial>
+        <inertial>
             <mass value="5" />
             <origin rpy="0 0 0" xyz="0 0 0" />
@@ -88,5 +88,5 @@
             </geometry>
         </collision>
-<inertial>
+        <inertial>
             <mass value="4" />
             <origin rpy="0 0 0" xyz="0 0 0" />
@@ -110,5 +110,5 @@
             </geometry>
         </collision>
-<inertial>
+        <inertial>
             <mass value="5" />
             <origin rpy="0 0 0" xyz="0 0 0" />
@@ -132,5 +132,5 @@
             </geometry>
         </collision>
-<inertial>
+        <inertial>
             <mass value="1.5" />
             <origin rpy="0 0 0" xyz="0 0 0" />
@@ -154,5 +154,5 @@
             </geometry>
         </collision>
-<inertial>
+        <inertial>
             <mass value="0.25" />
             <origin rpy="0 0 0" xyz="0 0 0" />
@@ -176,5 +176,5 @@
             </geometry>
         </collision>
-<inertial>
+        <inertial>
             <mass value="0.1" />
             <origin rpy="0 0 0" xyz="0 0 0" />
@@ -198,5 +198,5 @@
             </geometry>
         </collision>
-<inertial>
+        <inertial>
             <mass value="0.01" />
             <origin rpy="0 0 0" xyz="0 0 0" />
@@ -220,5 +220,5 @@
             </geometry>
         </collision>
-<inertial>
+        <inertial>
             <mass value="0.01" />
             <origin rpy="0 0 0" xyz="0 0 0" />
@@ -327,5 +327,5 @@
         <material>Gazebo/Grey</material>
     </gazebo>
-<transmission name="trans_joint_1">
+    <transmission name="trans_joint_1">
         <type>transmission_interface/SimpleTransmission</type>
         <joint name="joint_1">
@@ -412,3 +412,35 @@
         </plugin>
     </gazebo>
+    <gazebo reference="{prefix}link1">
+        <mu1>0.61</mu1>
+        <mu2>0.61</mu2>
+    </gazebo>
+    <gazebo reference="{prefix}link2">
+        <mu1>0.61</mu1>
+        <mu2>0.61</mu2>
+    </gazebo>
+    <gazebo reference="{prefix}link3">
+        <mu1>0.61</mu1>
+        <mu2>0.61</mu2>
+    </gazebo>
+    <gazebo reference="{prefix}link4">
+        <mu1>0.61</mu1>
+        <mu2>0.61</mu2>
+    </gazebo>
+    <gazebo reference="{prefix}link5">
+        <mu1>0.61</mu1>
+        <mu2>0.61</mu2>
+    </gazebo>
+    <gazebo reference="{prefix}link6">
+        <mu1>0.61</mu1>
+        <mu2>0.61</mu2>
+    </gazebo>
+    <gazebo reference="{prefix}left_finger">
+        <mu1>1.00</mu1>
+        <mu2>1.00</mu2>
+    </gazebo>
+    <gazebo reference="{prefix}right_finger">
+        <mu1>1.00</mu1>
+        <mu2>1.00</mu2>
+    </gazebo>
 </robot>

File: fanuc_ros/src/fanuc_lrmate200id_support/urdf/fanuc_lrmate200id_macro.xacro (robot description, xacro)
@@ -305,4 +305,36 @@
       <material>Gazebo/Grey</material>
     </gazebo>
+    <gazebo reference="{prefix}link1">
+      <mu1>0.61</mu1>
+      <mu2>0.61</mu2>
+    </gazebo>
+    <gazebo reference="{prefix}link2">
+      <mu1>0.61</mu1>
+      <mu2>0.61</mu2>
+    </gazebo>
+    <gazebo reference="{prefix}link3">
+      <mu1>0.61</mu1>
+      <mu2>0.61</mu2>
+    </gazebo>
+    <gazebo reference="{prefix}link4">
+      <mu1>0.61</mu1>
+      <mu2>0.61</mu2>
+    </gazebo>
+    <gazebo reference="{prefix}link5">
+      <mu1>0.61</mu1>
+      <mu2>0.61</mu2>
+    </gazebo>
+    <gazebo reference="{prefix}link6">
+      <mu1>0.61</mu1>
+      <mu2>0.61</mu2>
+    </gazebo>
+    <gazebo reference="{prefix}left_finger">
+      <mu1>1.00</mu1>
+      <mu2>1.00</mu2>
+    </gazebo>
+    <gazebo reference="{prefix}right_finger">
+      <mu1>1.00</mu1>
+      <mu2>1.00</mu2>
+    </gazebo>
   </xacro:macro>
 </robot>
