Commit message: Fanuc update.

File: rosbot_ros/src/rosbot/urdf/parameters.xacro (robot description, xacro)
@@ -36,3 +36,9 @@
     <xacro:property name="motor_damping" value="0.000" />
     <xacro:property name="motor_friction" value="0.00000" />
+    <material name="gray">
+        <color rgba="0.2 0.2 0.2 1"/>
+    </material>
+    <material name="green">
+        <color rgba="0.2 0.8 0.2 1"/>
+    </material>
 </robot>

File: rosbot_ros/src/rosbot/urdf/robot.xacro (robot description, xacro)
@@ -26,4 +26,5 @@
                 <box size="${base_size_x} ${base_size_y} ${base_size_z}"/>
             </geometry>
+            <material name="green"/>
         </visual>
         <!-- caster front -->
@@ -56,4 +57,5 @@
                 <sphere radius="${wheel_radius/2}"/>
             </geometry>
+            <material name="gray"/>
         </visual>
     </link>
@@ -92,4 +94,5 @@
                 <cylinder radius="${wheel_radius}" length="${wheel_width}"/>
             </geometry>
+            <material name="gray"/>
         </visual>
     </link>
@@ -136,4 +139,5 @@
                 <cylinder radius="${wheel_radius}" length="${wheel_width}"/>
             </geometry>
+            <material name="gray"/>
         </visual>
     </link>
